Commit message: Fixed the physics of the table and the geometry of the cup and cover. Spawned successfully in environment. Next step is to get the arm to pick up the cover and take it off the cup

File: environment/models/cup_with_cover/cover_model.urdf (robot description, URDF)
Before this commit: robot cover, 1 links, 0 joints
Links:
- link base_link: geometry collision cylinder length=0.02 radius=0.03; visual cylinder length=0.02 radius=0.03

File: environment/models/cup_with_cover/cup_model.urdf (robot description, URDF)
Before this commit: robot cup, 1 links, 0 joints
Links:
- link base_link: geometry collision cylinder length=0.10 radius=0.03; visual cylinder length=0.10 radius=0.03

Commit message: mid way through changes

File: environment/models/cup_with_cover/cover_model.urdf (robot description, URDF)
Before this commit: robot cover, 1 links, 0 joints
Links:
- link base_link: mass 5 -> 1; geometry collision box size=0.05 0.05 0.03; visual box size=0.05 0.05 0.03

File: environment/models/cup_with_cover/cup_model.urdf (robot description, URDF)
Before this commit: robot cup, 1 links, 0 joints
Links:
- link base_link: mass 10 -> 1; geometry collision box size=0.05 0.05 0.08; visual box size=0.05 0.05 0.08
